Commit message: all code cleaned up

File: ranger_description/models/urdf/ranger_mini.urdf (robot description, URDF)
Before this commit: robot ranger_mini_v2, 10 links, 9 joints
Links:
- added link base_footprint
Joints:
- added joint base_joint: type fixed, parent base_link, child base_footprint, origin xyz=0.0 0.0 -0.3 rpy=0 0 0
